Commit message: Robot spawn in gazebo successfully

File: ros2_ws/src/my_robot_description/urdf/common_properties.xacro (robot description, xacro)
@@ -1,19 +1,17 @@
 <?xml version="1.0"?>
 <robot xmlns:xacro="http://www.ros.org/wiki/xacro">
-    <material name="green">
-        <color rgba="0.0 0.5 0.0 1.0"/>
-    </material>
     <material name="blue">
-        <color rgba="0.0 0.0 0.5 1.0"/>
+        <color rgba="0 0 0.5 1" />
     </material>
     <material name="grey">
-        <color rgba="0.0 0.5 0.5 1.0"/>
+        <color rgba="0.5 0.5 0.5 1" />
     </material>
-    <xacro:macro name="box_inertia" params="m l w h xyz rpy ">
+    <xacro:macro name="box_inertia" params="m l w h xyz rpy">
         <inertial>
-            <origin xyz="${xyz}" rpy="${rpy}"/>
-            <mass value="${m}"/>
-            <inertia ixx="${(m/12) * (h*h + l*l)}" ixy="0.0" ixz="0.0"
-                     iyy="${(m/12) * (w*w + l*l)}"  iyz="0.0" izz="${(m/12) * (w*w + h*h)}" />
+            <origin xyz="${xyz}" rpy="${rpy}" />
+            <mass value="${m}" />
+            <inertia ixx="${(m/12) * (h*h + l*l)}" ixy="0" ixz="0"
+                     iyy="${(m/12) * (w*w + l*l)}" iyz="0"
+                     izz="${(m/12) * (w*w + h*h)}" />
         </inertial>
     </xacro:macro>

File: ros2_ws/src/my_robot_description/urdf/mobile_base.xacro (robot description, xacro)
@@ -6,13 +6,12 @@
     <xacro:property name="wheel_radius" value="0.1" />
     <xacro:property name="wheel_length" value="0.05" />
-    <link name="base_footprint">
-    </link>
+    <link name="base_footprint" />
     <link name="base_link">
         <visual>
             <geometry>
-                <box size="${base_length} ${base_width} ${base_height}"/>
+                <box size="${base_length} ${base_width} ${base_height}" />
             </geometry>
-            <origin xyz="0 0 ${base_height/2.0}" rpy="0 0 0"/>
-            <material name="blue"/>
+            <origin xyz="0 0 ${base_height / 2.0}" rpy="0 0 0" />
+            <material name="blue" />
         </visual>
         <collision>
@@ -23,5 +22,5 @@
         </collision>
         <xacro:box_inertia m="5.0" l="${base_length}" w="${base_width}" h="${base_height}"
-                            xyz="0 0 ${base_height/2.0}" rpy="0 0 0" />
+                           xyz="0 0 ${base_height / 2.0}" rpy="0 0 0" />
     </link>
     <xacro:macro name="wheel_link" params="prefix">
@@ -29,10 +28,8 @@
             <visual>
                 <geometry>
-                    <cylinder radius= "${wheel_radius}" length="${wheel_length}"/>
-                 </geometry>
-                <origin xyz="0.0 0.0 0.0" rpy="${pi/2.0} 0.0 0.0"/>
-                <material name="grey"/>
-                <xacro:cylinder_inertia m="1.0" r="${wheel_radius}" h="${wheel_length}"
-                                        xyz="0 0 0" rpy="${pi/2.0} 0.0 0.0" />
+                    <cylinder radius="${wheel_radius}" length="${wheel_length}" />
+                </geometry>
+                <origin xyz="0 0 0" rpy="${pi / 2.0} 0 0" />
+                <material name="grey" />
             </visual>
             <collision>
@@ -42,15 +39,17 @@
                 <origin xyz="0.0 0.0 0.0" rpy="${pi/2.0} 0.0 0.0"/>
             </collision>
+            <xacro:cylinder_inertia m="1.0" r="${wheel_radius}" h="${wheel_length}"
+                                    xyz="0 0 0" rpy="${pi / 2.0} 0 0" />
         </link>
     </xacro:macro>
-    <xacro:wheel_link prefix="right"/>
-    <xacro:wheel_link prefix="left"/>
-     <link name="caster_wheel_link">
+    <xacro:wheel_link prefix="right" />
+    <xacro:wheel_link prefix="left" />
+    <link name="caster_wheel_link">
         <visual>
             <geometry>
-                <sphere radius="${wheel_radius/2.0}"/>
+                <sphere radius="${wheel_radius / 2.0}" />
             </geometry>
-            <origin xyz="0.0 0.0 0.0" rpy="0.0 0.0 0.0"/>
-            <material name="grey"/>
+            <origin xyz="0 0 0" rpy="0 0 0" />
+            <material name="grey" />
         </visual>
         <collision>
@@ -64,24 +63,24 @@
     </link>
     <joint name="base_joint" type="fixed">
-        <origin xyz="0.0 0.0 ${wheel_radius}" rpy="0 0 0"/>
-        <parent link="base_footprint"/>
-        <child link="base_link"/>
+        <parent link="base_footprint" />
+        <child link="base_link" />
+        <origin xyz="0 0 ${wheel_radius}" rpy="0 0 0"/>
     </joint>
     <joint name="base_right_wheel_joint" type="continuous">
-        <origin xyz="${-base_length / 4.0} ${-(base_width + wheel_length)/2.0} 0.0" rpy="0 0 0"/>
-        <parent link="base_link"/>
-        <child link="right_wheel_link"/>
-        <axis xyz="0.0 1.0 0.0"/>
+        <parent link="base_link" />
+        <child link="right_wheel_link" />
+        <origin xyz="${-base_length / 4.0} ${-(base_width + wheel_length) / 2.0} 0" rpy="0 0 0" />
+        <axis xyz="0 1 0" />
     </joint>
     <joint name="base_left_wheel_joint" type="continuous">
-        <origin xyz="${-base_length / 4.0} ${(base_width + wheel_length)/2.0} 0.0" rpy="0 0 0"/>
-        <parent link="base_link"/>
-        <child link="left_wheel_link"/>
-        <axis xyz="0.0 1.0 0.0"/>
+        <parent link="base_link" />
+        <child link="left_wheel_link" />
+        <origin xyz="${-base_length / 4.0} ${(base_width + wheel_length) / 2.0} 0" rpy="0 0 0" />
+        <axis xyz="0 1 0" />
     </joint>
     <joint name="base_caster_wheel_joint" type="fixed">
-        <origin xyz="${base_length/3} 0.0 ${-wheel_radius/2.0}" rpy="0.0 0.0 0.0"/>
-        <parent link="base_link"/>
-        <child link="caster_wheel_link"/>
+        <parent link="base_link" />
+        <child link="caster_wheel_link" />
+        <origin xyz="${base_length / 3.0} 0 ${-wheel_radius / 2.0}" rpy="0 0 0" />
     </joint>
 </robot>

Commit message: V1 All working Alhamdullah

File: ros2_ws/src/my_robot_description/urdf/common_properties.xacro (robot description, xacro)
@@ -2,8 +2,14 @@
 <robot xmlns:xacro="http://www.ros.org/wiki/xacro">
     <material name="blue">
-        <color rgba="0 0 0.5 1" />
+        <color rgba="0.11 0.004 0.231 1" />
+    </material>
+    <material name="white">
+        <color rgba="0.984 0.98 0.988 1" />
     </material>
     <material name="grey">
         <color rgba="0.5 0.5 0.5 1" />
+    </material>
+    <material name="black">
+        <color rgba="0.05 0.1 0.1 1" />
     </material>
     <xacro:macro name="box_inertia" params="m l w h xyz rpy">

File: ros2_ws/src/my_robot_description/urdf/mobile_base.xacro (robot description, xacro)
@@ -3,5 +3,5 @@
     <xacro:property name="base_length" value="0.6" />
     <xacro:property name="base_width" value="0.4" />
-    <xacro:property name="base_height" value="0.2" />
+    <xacro:property name="base_height" value="0.15" />
     <xacro:property name="wheel_radius" value="0.1" />
     <xacro:property name="wheel_length" value="0.05" />
@@ -13,5 +13,5 @@
             </geometry>
             <origin xyz="0 0 ${base_height / 2.0}" rpy="0 0 0" />
-            <material name="blue" />
+            <material name="white" />
         </visual>
         <collision>
@@ -31,5 +31,5 @@
                 </geometry>
                 <origin xyz="0 0 0" rpy="${pi / 2.0} 0 0" />
-                <material name="grey" />
+                <material name="black" />
             </visual>
             <collision>
@@ -43,24 +43,28 @@
         </link>
     </xacro:macro>
-    <xacro:wheel_link prefix="right" />
-    <xacro:wheel_link prefix="left" />
-    <link name="caster_wheel_link">
-        <visual>
-            <geometry>
-                <sphere radius="${wheel_radius / 2.0}" />
-            </geometry>
-            <origin xyz="0 0 0" rpy="0 0 0" />
-            <material name="grey" />
-        </visual>
-        <collision>
-            <geometry>
-                <sphere radius="${wheel_radius/2.0}"/>
-            </geometry>
-            <origin xyz="0.0 0.0 0.0" rpy="0.0 0.0 0.0"/>
-        </collision>
-        <xacro:sphere_inertia m="0.5" r="${2*wheel_radius / 2.0}"
-                              xyz="0 0 0" rpy="0 0 0" />
-                              <!-- Multiplied by 2 to increase inertia -->
-    </link>
+    <xacro:wheel_link prefix="right_aft" />
+    <xacro:wheel_link prefix="left_aft" />
+    <xacro:wheel_link prefix="left_forward" />
+    <xacro:wheel_link prefix="right_forward" />
+    <!--
+        <link name="caster_wheel_link">
+            <visual>
+                <geometry>
+                    <sphere radius="${wheel_radius / 2.0}" />
+                </geometry>
+                <origin xyz="0 0 0" rpy="0 0 0" />
+                <material name="grey" />
+            </visual>
+            <collision>
+                <geometry>
+                    <sphere radius="${wheel_radius/2.0}"/>
+                </geometry>
+                <origin xyz="0.0 0.0 0.0" rpy="0.0 0.0 0.0"/>
+            </collision>
+            <xacro:sphere_inertia m="0.5" r="${2*wheel_radius / 2.0}"
+                                  xyz="0 0 0" rpy="0 0 0" />
+        </link>
+    -->
+   <!-- Multiplied by 2 to increase inertia -->
     <joint name="base_joint" type="fixed">
         <parent link="base_footprint" />
@@ -68,16 +72,29 @@
         <origin xyz="0 0 ${wheel_radius}" rpy="0 0 0"/>
     </joint>
-    <joint name="base_right_wheel_joint" type="continuous">
+    <joint name="base_right_aft_wheel_joint" type="continuous">
         <parent link="base_link" />
-        <child link="right_wheel_link" />
+        <child link="right_aft_wheel_link" />
         <origin xyz="${-base_length / 4.0} ${-(base_width + wheel_length) / 2.0} 0" rpy="0 0 0" />
         <axis xyz="0 1 0" />
     </joint>
-    <joint name="base_left_wheel_joint" type="continuous">
+    <joint name="base_right_forward_wheel_joint" type="continuous">
         <parent link="base_link" />
-        <child link="left_wheel_link" />
+        <child link="right_forward_wheel_link" />
+        <origin xyz="${base_length / 4.0} ${-(base_width + wheel_length) / 2.0} 0" rpy="0 0 0" />
+        <axis xyz="0 1 0" />
+    </joint>
+    <joint name="base_left_aft_wheel_joint" type="continuous">
+        <parent link="base_link" />
+        <child link="left_aft_wheel_link" />
         <origin xyz="${-base_length / 4.0} ${(base_width + wheel_length) / 2.0} 0" rpy="0 0 0" />
         <axis xyz="0 1 0" />
     </joint>
+    <joint name="base_left_forward_wheel_joint" type="continuous">
+        <parent link="base_link" />
+        <child link="left_forward_wheel_link" />
+        <origin xyz="${base_length / 4.0} ${(base_width + wheel_length) / 2.0} 0" rpy="0 0 0" />
+        <axis xyz="0 1 0" />
+    </joint>
+    <!--
     <joint name="base_caster_wheel_joint" type="fixed">
         <parent link="base_link" />
@@ -85,3 +102,4 @@
         <origin xyz="${base_length / 3.0} 0 ${-wheel_radius / 2.0}" rpy="0 0 0" />
     </joint>
+    -->
 </robot>
